Commit message: Updated robot xacro to use parameters from diff_params.yaml

File: nuturtle_description/urdf/turtlebot3_burger.urdf.xacro (robot description, xacro)
@@ -7,4 +7,13 @@
   -->
   <!-- <xacro:include filename="$(find turtlebot3_description)/urdf/common_properties.urdf"/> -->
+  <!--PROPERTIES-->
+  <!-- Get the path to the yaml file relative to the package -->
+  <xacro:property name="yaml_file" value="$(find nuturtle_description)/config/diff_params.yaml" />
+  <!-- load values from yaml file which are stored in a dictionary called props-->
+  <xacro:property name="props" value="${xacro.load_yaml(yaml_file)['/**']['ros__parameters']}" />
+  <!-- access individual properties -->
+  <xacro:property name="wheel_radius"  value="${props['wheel_radius']}" />
+  <xacro:property name="track_width"  value="${props['track_width']}" />
+  <xacro:property name="collision_radius"  value="${props['collision_radius']}" />
   <!-- Init colour -->
   <material name="black">
@@ -55,5 +64,10 @@
       <origin xyz="-0.032 0 0.070" rpy="0 0 0"/>
       <geometry>
-        <box size="0.140 0.140 0.143"/>
+        <xacro:if value="${collision_radius &lt; 0}">
+          <box size="0.140 0.140 0.143"/>
+        </xacro:if>
+        <xacro:unless value="${collision_radius &lt; 0}">
+          <cylinder length="0.143" radius="${collision_radius}"/>
+        </xacro:unless>
       </geometry>
     </collision>
@@ -67,5 +81,5 @@
     <parent link="base_link"/>
     <child link="wheel_left_link"/>
-    <origin xyz="0.0 0.08 0.023" rpy="-1.57 0 0"/>
+    <origin xyz="0.0 ${track_width / 2.} 0.023" rpy="-1.57 0 0"/>
     <axis xyz="0 0 1"/>
   </joint>
@@ -81,5 +95,5 @@
       <origin xyz="0 0 0" rpy="0 0 0"/>
       <geometry>
-        <cylinder length="0.018" radius="0.033"/>
+        <cylinder length="0.018" radius="${wheel_radius}"/>
       </geometry>
     </collision>
@@ -93,5 +107,5 @@
     <parent link="base_link"/>
     <child link="wheel_right_link"/>
-    <origin xyz="0.0 -0.080 0.023" rpy="-1.57 0 0"/>
+    <origin xyz="0.0 ${-track_width / 2.} 0.023" rpy="-1.57 0 0"/>
     <axis xyz="0 0 1"/>
   </joint>
@@ -107,5 +121,5 @@
       <origin xyz="0 0 0" rpy="0 0 0"/>
       <geometry>
-        <cylinder length="0.018" radius="0.033"/>
+        <cylinder length="0.018" radius="${wheel_radius}"/>
       </geometry>
     </collision>

Commit message: Modified xacro file to accept a color argument

File: nuturtle_description/urdf/turtlebot3_burger.urdf.xacro (robot description, xacro)
@@ -7,5 +7,7 @@
   -->
   <!-- <xacro:include filename="$(find turtlebot3_description)/urdf/common_properties.urdf"/> -->
-  <!--PROPERTIES-->
+  <!-- ARGUMENTS -->
+  <xacro:arg name="color" default="purple"/>
+  <!-- PROPERTIES -->
   <!-- Get the path to the yaml file relative to the package -->
   <xacro:property name="yaml_file" value="$(find nuturtle_description)/config/diff_params.yaml" />
@@ -17,4 +19,7 @@
   <xacro:property name="collision_radius"  value="${props['collision_radius']}" />
   <!-- Init colour -->
+  <material name="purple">
+    <color rgba= "0.3 0.16 0.52 1.0" />
+  </material>
   <material name="black">
       <color rgba="0.0 0.0 0.0 1.0"/>
@@ -59,5 +64,5 @@
         <mesh filename="package://nuturtle_description/meshes/burger_base.stl" scale="0.001 0.001 0.001"/>
       </geometry>
-      <material name="light_black"/>
+      <material name="$(arg color)"/>
     </visual>
     <collision>
